Commit message: move_group_interface学习

File: widowx_arm_description/urdf/widowx.urdf.xacro (robot description, xacro)
@@ -131,66 +131,4 @@
          </inertial>
       </link>
-      <!--link name="${prefix}gripper_rail_link">
-         <visual>
-            <origin xyz="0 0 0" rpy="0 0 1.57" />
-            <geometry>
-               <mesh filename="package://widowx_arm_description/meshes/gripper_rail_link.stl"/>
-            </geometry>
-            <xacro:material_black />
-         </visual>
-         <collision>
-            <origin xyz="0 0 0" rpy="0 0 0" />
-            <geometry>
-               <mesh filename="package://widowx_arm_description/meshes/gripper_rail_link.stl"/>
-            </geometry>
-         </collision>
-         <inertial>
-            <origin xyz="0 0 0" rpy="0 0 0" />
-            <mass value="1" />
-            <inertia ixx="1.0" ixy="0.0" ixz="0.0" iyy="1.0" iyz="0.0" izz="1.0" />
-         </inertial>
-      </link-->
-      <!--link name="${prefix}gripper_aux_link">
-      </link-->
-      <!--link name="${prefix}gripper_1_link">
-         <visual>
-            <origin xyz="0 -0.0007 0" rpy="0 0 1.57" />
-            <geometry>
-               <mesh filename="package://widowx_arm_description/meshes/gripper_hand_fixed_link.stl"/>
-            </geometry>
-            <xacro:material_black />
-         </visual>
-         <collision>
-            <origin xyz="0 0 0" rpy="0 0 0" />
-            <geometry>
-               <mesh filename="package://widowx_arm_description/meshes/gripper_hand_fixed_link.stl"/>
-            </geometry>
-         </collision>
-         <inertial>
-            <origin xyz="0 0 0" rpy="0 0 0" />
-            <mass value="1" />
-            <inertia ixx="1.0" ixy="0.0" ixz="0.0" iyy="1.0" iyz="0.0" izz="1.0" />
-         </inertial>
-      </link>
-      <link name="${prefix}gripper_2_link">
-         <visual>
-            <origin xyz="0 0.0007 0" rpy="0 0 -1.57" />
-            <geometry>
-               <mesh filename="package://widowx_arm_description/meshes/gripper_hand_fixed_link.stl"/>
-            </geometry>
-            <xacro:material_black />
-         </visual>
-         <collision>
-            <origin xyz="0 0 0" rpy="0 0 0" />
-            <geometry>
-               <mesh filename="package://widowx_arm_description/meshes/gripper_hand_fixed_link.stl"/>
-            </geometry>
-         </collision>
-         <inertial>
-            <origin xyz="0 0 0" rpy="0 0 0" />
-            <mass value="1" />
-            <inertia ixx="1.0" ixy="0.0" ixz="0.0" iyy="1.0" iyz="0.0" izz="1.0" />
-         </inertial>
-      </link-->
       <!-- joints -->
       <joint name="${prefix}arm_base_joint" type="fixed">
@@ -235,43 +173,6 @@
          <limit lower="-2.617" upper="2.617" effort="6" velocity="1.571" />
       </joint>
-      <!--joint name="${prefix}joint_6" type="fixed">
-         <origin xyz = "0 0 ${M_SCALE*43}" rpy="0 0 0" />
-         <parent link="${prefix}wrist_2_link" />
-         <child link="${prefix}gripper_rail_link" />
-         <axis xyz="0 0 1" />
-         <limit lower="-0.31" upper="0.1" effort="6" velocity="0.5" />
-      </joint-->
-      <!--joint name="${prefix}gripper_revolute_joint" type="revolute">
-         <origin xyz = "0 0 0.065" rpy="0 0 0" />
-         <parent link="${prefix}wrist_2_link" />
-         <child link="${prefix}gripper_aux_link" />
-         <axis xyz="0 0 1" />
-         <limit lower="-2.6" upper="2.6" effort="6" velocity="0.5" />
-      </joint-->
-      <!--joint name="${prefix}gripper_prismatic_joint_1" type="prismatic">
-         <origin xyz="0 0 0" rpy="0 0 0" />
-         <parent link="${prefix}gripper_rail_link" />
-         <child link="${prefix}gripper_1_link" />
-         <axis xyz="0 -1 0" />
-         <limit lower="0" upper="0.027" effort="6" velocity="0.5" />
-      </joint>
-      <joint name="${prefix}gripper_prismatic_joint_2" type="prismatic">
-         <origin xyz="0 0 0" rpy="0 0 0" />
-         <parent link="${prefix}gripper_rail_link" />
-         <child link="${prefix}gripper_2_link" />
-         <mimic joint="${prefix}gripper_prismatic_joint_1" />
-         <axis xyz="0 1 0" />
-         <limit lower="0" upper="0.027" effort="6" velocity="0.5" />
-      </joint-->
       <!-- gripper -->
   <xacro:include filename="$(find widowx_arm_description)/urdf/widowx_gripper.xacro"/>
-  <!--link name="gripper_link"/>
-    <joint name="gripper_link_joint" type="revolute">
-      <origin xyz="0 0 0.110" rpy="0 0 0"/>
-      <parent link="${prefix}wrist_1_link" />
-      <child link="gripper_link"/>
-      <limit effort="6" velocity="1" lower="-3.14" upper="3.14"/>
-      <axis xyz="1 0 0"/>
-    </joint-->
    </xacro:macro>
   <transmission name="tran1">
@@ -309,5 +210,5 @@
  <transmission name="tran5">
     <type>transmission_interface/SimpleTransmission</type>
-    <joint name="joint_6"/>
+    <joint name="joint_5"/>
     <actuator name="motor5">
       <hardwareInterface>EffortJointInterface</hardwareInterface>
@@ -317,5 +218,5 @@
  <transmission name="tran6">
     <type>transmission_interface/SimpleTransmission</type>
-    <joint name="gripper_prismatic_joint_1"/>
+    <joint name="gripper_joint"/>
     <actuator name="motor6">
       <hardwareInterface>EffortJointInterface</hardwareInterface>

File: widowx_arm_description/urdf/widowx_gripper.xacro (robot description, xacro)
@@ -1,3 +1,3 @@
-<?xml version="1.0"?>
+<?xml version="1.0" encoding="UTF-8"?>
 <robot xmlns:xacro="http://ros.org/wiki/xacro">
    <link name="${prefix}gripper_rail_link">
